File: stav-keeb-65.kicad_pcb (KiCad board)
At the start: 2 copper layers, 346 parts, among them SW1 DRV5055A4QDBZR, SW10 DRV5055A4QDBZR, SW11 DRV5055A4QDBZR, SW12 DRV5055A4QDBZR, SW13 DRV5055A4QDBZR, SW14 DRV5055A4QDBZR, SW15 DRV5055A4QDBZR, SW16 DRV5055A4QDBZR, SW17 DRV5055A4QDBZR, SW18 DRV5055A4QDBZR, SW19 DRV5055A4QDBZR, SW2 DRV5055A4QDBZR, SW20 DRV5055A4QDBZR, SW21 DRV5055A4QDBZR, SW22 DRV5055A4QDBZR, SW23 DRV5055A4QDBZR, SW24 DRV5055A4QDBZR, SW25 DRV5055A4QDBZR, SW26 DRV5055A4QDBZR, SW27 DRV5055A4QDBZR, SW28 DRV5055A4QDBZR, SW29 DRV5055A4QDBZR, SW3 DRV5055A4QDBZR, SW30 DRV5055A4QDBZR, SW31 DRV5055A4QDBZR, SW32 DRV5055A4QDBZR, SW33 DRV5055A4QDBZR, SW34 DRV5055A4QDBZR, SW35 DRV5055A4QDBZR, SW36 DRV5055A4QDBZR, SW37 DRV5055A4QDBZR, SW38 DRV5055A4QDBZR, SW39 DRV5055A4QDBZR, SW4 DRV5055A4QDBZR, SW40 DRV5055A4QDBZR, SW41 DRV5055A4QDBZR, SW42 DRV5055A4QDBZR, SW43 DRV5055A4QDBZR, SW44 DRV5055A4QDBZR, SW45 DRV5055A4QDBZR, SW46 DRV5055A4QDBZR, SW47 DRV5055A4QDBZR, SW48 DRV5055A4QDBZR, SW49 DRV5055A4QDBZR, SW5 DRV5055A4QDBZR, SW50 DRV5055A4QDBZR, SW51 DRV5055A4QDBZR, SW52 DRV5055A4QDBZR, SW53 DRV5055A4QDBZR, SW54 DRV5055A4QDBZR, SW55 DRV5055A4QDBZR, SW56 DRV5055A4QDBZR, SW57 DRV5055A4QDBZR, SW58 DRV5055A4QDBZR, SW59 DRV5055A4QDBZR, SW6 DRV5055A4QDBZR, SW60 DRV5055A4QDBZR, SW61 DRV5055A4QDBZR, SW62 DRV5055A4QDBZR, SW63 DRV5055A4QDBZR, SW64 DRV5055A4QDBZR, SW65 DRV5055A4QDBZR, SW66 DRV5055A4QDBZR, SW67 DRV5055A4QDBZR, SW68 DRV5055A4QDBZR, SW69 DRV5055A4QDBZR, SW7 DRV5055A4QDBZR, SW70 DRV5055A4QDBZR, SW71 DRV5055A4QDBZR, SW72 DRV5055A4QDBZR, SW73 DRV5055A4QDBZR, SW74 DRV5055A4QDBZR, SW75 DRV5055A4QDBZR, SW76 DRV5055A4QDBZR, SW77 DRV5055A4QDBZR, SW78 DRV5055A4QDBZR, SW79 DRV5055A4QDBZR, SW8 DRV5055A4QDBZR, SW80 DRV5055A4QDBZR, SW9 DRV5055A4QDBZR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

Commit message: some more schematic fixes
Parts:
- removed C100, C101, C102, C103, C104, C105, C106, C107, C109, C111, C112, C116, C119, C120, C127, C129, C135, C54, C55, C56, C57, C58, C59, C60, C61, C62, C63, C64, C65, C67, C68, C69, C70, C73, C74, C75, C76, C77, C78, C79, C80, C81, C82, C83, C84, C85, C87, C88, C89, C90, C93, C94, C95, C96, C97, C98, C99: 100nF, Capacitor_SMD:C_0603_1608Metric_Pad1.08x0.95mm_HandSolder
- removed C108, C110, C115, C126, C130, C131, C132, C133, C134, C66, C71, C72, C86, C91, C92: 1uF, Capacitor_SMD:C_0603_1608Metric_Pad1.08x0.95mm_HandSolder
- removed C113, C114: 33pF, Capacitor_SMD:C_0603_1608Metric_Pad1.08x0.95mm_HandSolder
- removed C117, C118, C128: 10uF, Capacitor_SMD:C_1206_3216Metric_Pad1.33x1.80mm_HandSolder
- removed C121: 22uF, Capacitor_SMD:C_1206_3216Metric_Pad1.33x1.80mm_HandSolder
- removed C122: 4.7nF, Capacitor_SMD:C_0603_1608Metric_Pad1.08x0.95mm_HandSolder
- removed C123, C124: 1nF, Capacitor_SMD:C_0603_1608Metric_Pad1.08x0.95mm_HandSolder
- removed C125: 10nF, Capacitor_SMD:C_0603_1608Metric_Pad1.08x0.95mm_HandSolder
- removed R100, R95, R97, R98, R99: 0, Resistor_SMD:R_0603_1608Metric_Pad0.98x0.95mm_HandSolder
- removed R101, R113: 1k, Resistor_SMD:R_0603_1608Metric_Pad0.98x0.95mm_HandSolder
- removed R102, R114, R96: 10k, Resistor_SMD:R_0603_1608Metric_Pad0.98x0.95mm_HandSolder
- removed R103, R104: 5.1k, Resistor_SMD:R_0603_1608Metric_Pad0.98x0.95mm_HandSolder
- removed R105: 1M, Resistor_SMD:R_0603_1608Metric_Pad0.98x0.95mm_HandSolder
- removed R106, R107: 100k, Resistor_SMD:R_0603_1608Metric_Pad0.98x0.95mm_HandSolder
- removed R108, R109: 22, Resistor_SMD:R_0603_1608Metric_Pad0.98x0.95mm_HandSolder
- removed R110: 10, Resistor_SMD:R_0603_1608Metric_Pad0.98x0.95mm_HandSolder
- removed R111, R112: 10k 0.1%, Resistor_SMD:R_0603_1608Metric_Pad0.98x0.95mm_HandSolder
- removed SW10, SW11, SW12, SW13, SW14, SW15, SW16, SW17, SW18, SW19, SW20, SW21, SW22, SW23, SW24, SW25, SW26, SW27, SW28, SW29, SW30, SW31, SW32, SW33, SW34, SW35, SW36, SW37, SW38, SW39, SW4, SW40, SW41, SW42, SW43, SW44, SW45, SW46, SW47, SW48, SW49, SW5, SW50, SW51, SW52, SW53, SW54, SW55, SW56, SW57, SW58, SW59, SW6, SW60, SW61, SW62, SW63, SW64, SW65, SW66, SW67, SW68, SW69, SW7, SW70, SW71, SW72, SW73, SW74, SW75, SW76, SW77, SW78, SW79, SW8, SW80, SW9: DRV5055A4QDBZR, easyeda2kicad:SOT-23-3_L2.9-W1.3-P1.90-LS2.4-BR
- removed U9: OPA320AIDBVR, easyeda2kicad:SOT-23-5_L3.0-W1.7-P0.95-LS2.8-BR
- removed _SW201: RESET, easyeda2kicad:SW-SMD_4P-L5.1-W5.1-P3.70-LS6.5-TL_H1.5
- removed _SW202: BOOTSEL, easyeda2kicad:SW-SMD_4P-L5.1-W5.1-P3.70-LS6.5-TL_H1.5
- added K_C1: 100nF, Capacitor_SMD:C_0603_1608Metric_Pad1.08x0.95mm_HandSolder, B.Cu at (38.1, 38.1)
- added K_C10: 100nF, Capacitor_SMD:C_0603_1608Metric_Pad1.08x0.95mm_HandSolder, B.Cu at (209.6, 38.1)
- added K_C11: 100nF, Capacitor_SMD:C_0603_1608Metric_Pad1.08x0.95mm_HandSolder, B.Cu at (228.6, 38.1)
- added K_C12: 100nF, Capacitor_SMD:C_0603_1608Metric_Pad1.08x0.95mm_HandSolder, B.Cu at (247.7, 38.1)
- added K_C13: 100nF, Capacitor_SMD:C_0603_1608Metric_Pad1.08x0.95mm_HandSolder, B.Cu at (266.7, 38.1)
- added K_C14: 100nF, Capacitor_SMD:C_0603_1608Metric_Pad1.08x0.95mm_HandSolder, B.Cu at (295.3, 38.1)
- added K_C15: 100nF, Capacitor_SMD:C_0603_1608Metric_Pad1.08x0.95mm_HandSolder, B.Cu at (42.9, 57.1)
- added K_C16: 100nF, Capacitor_SMD:C_0603_1608Metric_Pad1.08x0.95mm_HandSolder, B.Cu at (66.7, 57.1)
- added K_C17: 100nF, Capacitor_SMD:C_0603_1608Metric_Pad1.08x0.95mm_HandSolder, B.Cu at (85.7, 57.1)
- added K_C18: 100nF, Capacitor_SMD:C_0603_1608Metric_Pad1.08x0.95mm_HandSolder, B.Cu at (104.8, 57.1)
- added K_C19: 100nF, Capacitor_SMD:C_0603_1608Metric_Pad1.08x0.95mm_HandSolder, B.Cu at (123.8, 57.1)
- added K_C2: 100nF, Capacitor_SMD:C_0603_1608Metric_Pad1.08x0.95mm_HandSolder, B.Cu at (57.1, 38.1)
- added K_C20: 100nF, Capacitor_SMD:C_0603_1608Metric_Pad1.08x0.95mm_HandSolder, B.Cu at (142.9, 57.1)
- added K_C21: 100nF, Capacitor_SMD:C_0603_1608Metric_Pad1.08x0.95mm_HandSolder, B.Cu at (161.9, 57.1)
- added K_C22: 100nF, Capacitor_SMD:C_0603_1608Metric_Pad1.08x0.95mm_HandSolder, B.Cu at (181.0, 57.1)
- added K_C23: 100nF, Capacitor_SMD:C_0603_1608Metric_Pad1.08x0.95mm_HandSolder, B.Cu at (200.0, 57.1)
- added K_C24: 100nF, Capacitor_SMD:C_0603_1608Metric_Pad1.08x0.95mm_HandSolder, B.Cu at (219.1, 57.1)
- added K_C25: 100nF, Capacitor_SMD:C_0603_1608Metric_Pad1.08x0.95mm_HandSolder, B.Cu at (238.1, 57.1)
- added K_C26: 100nF, Capacitor_SMD:C_0603_1608Metric_Pad1.08x0.95mm_HandSolder, B.Cu at (257.2, 57.1)
- added K_C27: 100nF, Capacitor_SMD:C_0603_1608Metric_Pad1.08x0.95mm_HandSolder, B.Cu at (276.2, 57.1)
- added K_C28: 100nF, Capacitor_SMD:C_0603_1608Metric_Pad1.08x0.95mm_HandSolder, B.Cu at (300.0, 57.1)
- added K_C29: 100nF, Capacitor_SMD:C_0603_1608Metric_Pad1.08x0.95mm_HandSolder, B.Cu at (45.2, 76.2)
- added K_C3: 100nF, Capacitor_SMD:C_0603_1608Metric_Pad1.08x0.95mm_HandSolder, B.Cu at (76.2, 38.1)
- added K_C30: 100nF, Capacitor_SMD:C_0603_1608Metric_Pad1.08x0.95mm_HandSolder, B.Cu at (71.4, 76.2)
- added K_C31: 100nF, Capacitor_SMD:C_0603_1608Metric_Pad1.08x0.95mm_HandSolder, B.Cu at (90.5, 76.2)
- added K_C32: 100nF, Capacitor_SMD:C_0603_1608Metric_Pad1.08x0.95mm_HandSolder, B.Cu at (109.5, 76.2)
- added K_C33: 100nF, Capacitor_SMD:C_0603_1608Metric_Pad1.08x0.95mm_HandSolder, B.Cu at (128.6, 76.2)
- added K_C34: 100nF, Capacitor_SMD:C_0603_1608Metric_Pad1.08x0.95mm_HandSolder, B.Cu at (147.6, 76.2)
- added K_C35: 100nF, Capacitor_SMD:C_0603_1608Metric_Pad1.08x0.95mm_HandSolder, B.Cu at (166.7, 76.2)
- added K_C36: 100nF, Capacitor_SMD:C_0603_1608Metric_Pad1.08x0.95mm_HandSolder, B.Cu at (185.7, 76.2)
- added K_C37: 100nF, Capacitor_SMD:C_0603_1608Metric_Pad1.08x0.95mm_HandSolder, B.Cu at (204.8, 76.2)
- added K_C38: 100nF, Capacitor_SMD:C_0603_1608Metric_Pad1.08x0.95mm_HandSolder, B.Cu at (223.8, 76.2)
- added K_C39: 100nF, Capacitor_SMD:C_0603_1608Metric_Pad1.08x0.95mm_HandSolder, B.Cu at (242.9, 76.2)
- added K_C4: 100nF, Capacitor_SMD:C_0603_1608Metric_Pad1.08x0.95mm_HandSolder, B.Cu at (95.2, 38.1)
- added K_C40: 100nF, Capacitor_SMD:C_0603_1608Metric_Pad1.08x0.95mm_HandSolder, B.Cu at (261.9, 76.2)
- added K_C41: 100nF, Capacitor_SMD:C_0603_1608Metric_Pad1.08x0.95mm_HandSolder, B.Cu at (292.9, 76.2)
- added K_C42: 100nF, Capacitor_SMD:C_0603_1608Metric_Pad1.08x0.95mm_HandSolder, B.Cu at (50.0, 95.2)
- added K_C43: 100nF, Capacitor_SMD:C_0603_1608Metric_Pad1.08x0.95mm_HandSolder, B.Cu at (81.0, 95.2)
- added K_C44: 100nF, Capacitor_SMD:C_0603_1608Metric_Pad1.08x0.95mm_HandSolder, B.Cu at (100.0, 95.2)
- added K_C45: 100nF, Capacitor_SMD:C_0603_1608Metric_Pad1.08x0.95mm_HandSolder, B.Cu at (119.1, 95.2)
- added K_C46: 100nF, Capacitor_SMD:C_0603_1608Metric_Pad1.08x0.95mm_HandSolder, B.Cu at (138.1, 95.2)
- added K_C47: 100nF, Capacitor_SMD:C_0603_1608Metric_Pad1.08x0.95mm_HandSolder, B.Cu at (157.2, 95.2)
- added K_C48: 100nF, Capacitor_SMD:C_0603_1608Metric_Pad1.08x0.95mm_HandSolder, B.Cu at (176.2, 95.2)
- added K_C49: 100nF, Capacitor_SMD:C_0603_1608Metric_Pad1.08x0.95mm_HandSolder, B.Cu at (195.3, 95.2)
- added K_C5: 100nF, Capacitor_SMD:C_0603_1608Metric_Pad1.08x0.95mm_HandSolder, B.Cu at (114.3, 38.1)
- added K_C50: 100nF, Capacitor_SMD:C_0603_1608Metric_Pad1.08x0.95mm_HandSolder, B.Cu at (214.3, 95.2)
- added K_C51: 100nF, Capacitor_SMD:C_0603_1608Metric_Pad1.08x0.95mm_HandSolder, B.Cu at (233.4, 95.2)
- added K_C52: 100nF, Capacitor_SMD:C_0603_1608Metric_Pad1.08x0.95mm_HandSolder, B.Cu at (252.4, 95.2)
- added K_C53: 100nF, Capacitor_SMD:C_0603_1608Metric_Pad1.08x0.95mm_HandSolder, B.Cu at (288.1, 95.2)
- added K_C54: 100nF, Capacitor_SMD:C_0603_1608Metric_Pad1.08x0.95mm_HandSolder, B.Cu at (40.5, 114.3)
- added K_C55: 100nF, Capacitor_SMD:C_0603_1608Metric_Pad1.08x0.95mm_HandSolder, B.Cu at (64.3, 114.3)
- added K_C56: 100nF, Capacitor_SMD:C_0603_1608Metric_Pad1.08x0.95mm_HandSolder, B.Cu at (88.1, 114.3)
- added K_C57: 100nF, Capacitor_SMD:C_0603_1608Metric_Pad1.08x0.95mm_HandSolder, B.Cu at (159.5, 114.3)
- added K_C58: 100nF, Capacitor_SMD:C_0603_1608Metric_Pad1.08x0.95mm_HandSolder, B.Cu at (231.0, 114.3)
- added K_C59: 100nF, Capacitor_SMD:C_0603_1608Metric_Pad1.08x0.95mm_HandSolder, B.Cu at (254.8, 114.3)
- added K_C6: 100nF, Capacitor_SMD:C_0603_1608Metric_Pad1.08x0.95mm_HandSolder, B.Cu at (133.3, 38.1)
- added K_C60: 100nF, Capacitor_SMD:C_0603_1608Metric_Pad1.08x0.95mm_HandSolder, B.Cu at (278.6, 114.3)
- added K_C61: 100nF, Capacitor_SMD:C_0603_1608Metric_Pad1.08x0.95mm_HandSolder, B.Cu at (302.4, 114.3)
- added K_C7: 100nF, Capacitor_SMD:C_0603_1608Metric_Pad1.08x0.95mm_HandSolder, B.Cu at (152.4, 38.1)
- added K_C8: 100nF, Capacitor_SMD:C_0603_1608Metric_Pad1.08x0.95mm_HandSolder, B.Cu at (171.4, 38.1)
- added K_C9: 100nF, Capacitor_SMD:C_0603_1608Metric_Pad1.08x0.95mm_HandSolder, B.Cu at (190.5, 38.1)
- added K_SW1: DRV5055A4QDBZR, easyeda2kicad:SOT-23-3_L2.9-W1.3-P1.90-LS2.4-BR, F.Cu at (38.1, 38.1)
- added K_SW10: DRV5055A4QDBZR, easyeda2kicad:SOT-23-3_L2.9-W1.3-P1.90-LS2.4-BR, F.Cu at (209.6, 38.1)
- added K_SW11: DRV5055A4QDBZR, easyeda2kicad:SOT-23-3_L2.9-W1.3-P1.90-LS2.4-BR, F.Cu at (228.6, 38.1)
- added K_SW12: DRV5055A4QDBZR, easyeda2kicad:SOT-23-3_L2.9-W1.3-P1.90-LS2.4-BR, F.Cu at (247.7, 38.1)
- added K_SW13: DRV5055A4QDBZR, easyeda2kicad:SOT-23-3_L2.9-W1.3-P1.90-LS2.4-BR, F.Cu at (266.7, 38.1)
- added K_SW14: DRV5055A4QDBZR, easyeda2kicad:SOT-23-3_L2.9-W1.3-P1.90-LS2.4-BR, F.Cu at (295.3, 38.1)
- added K_SW15: DRV5055A4QDBZR, easyeda2kicad:SOT-23-3_L2.9-W1.3-P1.90-LS2.4-BR, F.Cu at (42.9, 57.1)
- added K_SW16: DRV5055A4QDBZR, easyeda2kicad:SOT-23-3_L2.9-W1.3-P1.90-LS2.4-BR, F.Cu at (66.7, 57.1)
- added K_SW17: DRV5055A4QDBZR, easyeda2kicad:SOT-23-3_L2.9-W1.3-P1.90-LS2.4-BR, F.Cu at (85.7, 57.1)
- added K_SW18: DRV5055A4QDBZR, easyeda2kicad:SOT-23-3_L2.9-W1.3-P1.90-LS2.4-BR, F.Cu at (104.8, 57.1)
- added K_SW19: DRV5055A4QDBZR, easyeda2kicad:SOT-23-3_L2.9-W1.3-P1.90-LS2.4-BR, F.Cu at (123.8, 57.1)
- added K_SW2: DRV5055A4QDBZR, easyeda2kicad:SOT-23-3_L2.9-W1.3-P1.90-LS2.4-BR, F.Cu at (57.1, 38.1)
- added K_SW20: DRV5055A4QDBZR, easyeda2kicad:SOT-23-3_L2.9-W1.3-P1.90-LS2.4-BR, F.Cu at (142.9, 57.1)
- added K_SW21: DRV5055A4QDBZR, easyeda2kicad:SOT-23-3_L2.9-W1.3-P1.90-LS2.4-BR, F.Cu at (161.9, 57.1)
- added K_SW22: DRV5055A4QDBZR, easyeda2kicad:SOT-23-3_L2.9-W1.3-P1.90-LS2.4-BR, F.Cu at (181.0, 57.1)
- added K_SW23: DRV5055A4QDBZR, easyeda2kicad:SOT-23-3_L2.9-W1.3-P1.90-LS2.4-BR, F.Cu at (200.0, 57.1)
- added K_SW24: DRV5055A4QDBZR, easyeda2kicad:SOT-23-3_L2.9-W1.3-P1.90-LS2.4-BR, F.Cu at (219.1, 57.1)
- added K_SW25: DRV5055A4QDBZR, easyeda2kicad:SOT-23-3_L2.9-W1.3-P1.90-LS2.4-BR, F.Cu at (238.1, 57.1)
- added K_SW26: DRV5055A4QDBZR, easyeda2kicad:SOT-23-3_L2.9-W1.3-P1.90-LS2.4-BR, F.Cu at (257.2, 57.1)
- added K_SW27: DRV5055A4QDBZR, easyeda2kicad:SOT-23-3_L2.9-W1.3-P1.90-LS2.4-BR, F.Cu at (276.2, 57.1)
- added K_SW28: DRV5055A4QDBZR, easyeda2kicad:SOT-23-3_L2.9-W1.3-P1.90-LS2.4-BR, F.Cu at (300.0, 57.1)
- added K_SW29: DRV5055A4QDBZR, easyeda2kicad:SOT-23-3_L2.9-W1.3-P1.90-LS2.4-BR, F.Cu at (45.2, 76.2)
- added K_SW3: DRV5055A4QDBZR, easyeda2kicad:SOT-23-3_L2.9-W1.3-P1.90-LS2.4-BR, F.Cu at (76.2, 38.1)
- added K_SW30: DRV5055A4QDBZR, easyeda2kicad:SOT-23-3_L2.9-W1.3-P1.90-LS2.4-BR, F.Cu at (71.4, 76.2)
- added K_SW31: DRV5055A4QDBZR, easyeda2kicad:SOT-23-3_L2.9-W1.3-P1.90-LS2.4-BR, F.Cu at (90.5, 76.2)
- added K_SW32: DRV5055A4QDBZR, easyeda2kicad:SOT-23-3_L2.9-W1.3-P1.90-LS2.4-BR, F.Cu at (109.5, 76.2)
- added K_SW33: DRV5055A4QDBZR, easyeda2kicad:SOT-23-3_L2.9-W1.3-P1.90-LS2.4-BR, F.Cu at (128.6, 76.2)
- added K_SW34: DRV5055A4QDBZR, easyeda2kicad:SOT-23-3_L2.9-W1.3-P1.90-LS2.4-BR, F.Cu at (147.6, 76.2)
- added K_SW35: DRV5055A4QDBZR, easyeda2kicad:SOT-23-3_L2.9-W1.3-P1.90-LS2.4-BR, F.Cu at (166.7, 76.2)
- added K_SW36: DRV5055A4QDBZR, easyeda2kicad:SOT-23-3_L2.9-W1.3-P1.90-LS2.4-BR, F.Cu at (185.7, 76.2)
- added K_SW37: DRV5055A4QDBZR, easyeda2kicad:SOT-23-3_L2.9-W1.3-P1.90-LS2.4-BR, F.Cu at (204.8, 76.2)
- added K_SW38: DRV5055A4QDBZR, easyeda2kicad:SOT-23-3_L2.9-W1.3-P1.90-LS2.4-BR, F.Cu at (223.8, 76.2)
- added K_SW39: DRV5055A4QDBZR, easyeda2kicad:SOT-23-3_L2.9-W1.3-P1.90-LS2.4-BR, F.Cu at (242.9, 76.2)
- added K_SW4: DRV5055A4QDBZR, easyeda2kicad:SOT-23-3_L2.9-W1.3-P1.90-LS2.4-BR, F.Cu at (95.2, 38.1)
- added K_SW40: DRV5055A4QDBZR, easyeda2kicad:SOT-23-3_L2.9-W1.3-P1.90-LS2.4-BR, F.Cu at (261.9, 76.2)
- added K_SW41: DRV5055A4QDBZR, easyeda2kicad:SOT-23-3_L2.9-W1.3-P1.90-LS2.4-BR, F.Cu at (292.9, 76.2)
- added K_SW42: DRV5055A4QDBZR, easyeda2kicad:SOT-23-3_L2.9-W1.3-P1.90-LS2.4-BR, F.Cu at (50.0, 95.2)
- added K_SW43: DRV5055A4QDBZR, easyeda2kicad:SOT-23-3_L2.9-W1.3-P1.90-LS2.4-BR, F.Cu at (81.0, 95.2)
- added K_SW44: DRV5055A4QDBZR, easyeda2kicad:SOT-23-3_L2.9-W1.3-P1.90-LS2.4-BR, F.Cu at (100.0, 95.2)
- added K_SW45: DRV5055A4QDBZR, easyeda2kicad:SOT-23-3_L2.9-W1.3-P1.90-LS2.4-BR, F.Cu at (119.1, 95.2)
- added K_SW46: DRV5055A4QDBZR, easyeda2kicad:SOT-23-3_L2.9-W1.3-P1.90-LS2.4-BR, F.Cu at (138.1, 95.2)
- added K_SW47: DRV5055A4QDBZR, easyeda2kicad:SOT-23-3_L2.9-W1.3-P1.90-LS2.4-BR, F.Cu at (157.2, 95.2)
- added K_SW48: DRV5055A4QDBZR, easyeda2kicad:SOT-23-3_L2.9-W1.3-P1.90-LS2.4-BR, F.Cu at (176.2, 95.2)
- added K_SW49: DRV5055A4QDBZR, easyeda2kicad:SOT-23-3_L2.9-W1.3-P1.90-LS2.4-BR, F.Cu at (195.3, 95.2)
- added K_SW5: DRV5055A4QDBZR, easyeda2kicad:SOT-23-3_L2.9-W1.3-P1.90-LS2.4-BR, F.Cu at (114.3, 38.1)
- added K_SW50: DRV5055A4QDBZR, easyeda2kicad:SOT-23-3_L2.9-W1.3-P1.90-LS2.4-BR, F.Cu at (214.3, 95.2)
- added K_SW51: DRV5055A4QDBZR, easyeda2kicad:SOT-23-3_L2.9-W1.3-P1.90-LS2.4-BR, F.Cu at (233.4, 95.2)
- added K_SW52: DRV5055A4QDBZR, easyeda2kicad:SOT-23-3_L2.9-W1.3-P1.90-LS2.4-BR, F.Cu at (252.4, 95.2)
- added K_SW53: DRV5055A4QDBZR, easyeda2kicad:SOT-23-3_L2.9-W1.3-P1.90-LS2.4-BR, F.Cu at (288.1, 95.2)
- added K_SW54: DRV5055A4QDBZR, easyeda2kicad:SOT-23-3_L2.9-W1.3-P1.90-LS2.4-BR, F.Cu at (40.5, 114.3)
- added K_SW55: DRV5055A4QDBZR, easyeda2kicad:SOT-23-3_L2.9-W1.3-P1.90-LS2.4-BR, F.Cu at (64.3, 114.3)
- added K_SW56: DRV5055A4QDBZR, easyeda2kicad:SOT-23-3_L2.9-W1.3-P1.90-LS2.4-BR, F.Cu at (88.1, 114.3)
- added K_SW57: DRV5055A4QDBZR, easyeda2kicad:SOT-23-3_L2.9-W1.3-P1.90-LS2.4-BR, F.Cu at (159.5, 114.3)
- added K_SW58: DRV5055A4QDBZR, easyeda2kicad:SOT-23-3_L2.9-W1.3-P1.90-LS2.4-BR, F.Cu at (231.0, 114.3)
- added K_SW59: DRV5055A4QDBZR, easyeda2kicad:SOT-23-3_L2.9-W1.3-P1.90-LS2.4-BR, F.Cu at (254.8, 114.3)
- added K_SW6: DRV5055A4QDBZR, easyeda2kicad:SOT-23-3_L2.9-W1.3-P1.90-LS2.4-BR, F.Cu at (133.3, 38.1)
- added K_SW60: DRV5055A4QDBZR, easyeda2kicad:SOT-23-3_L2.9-W1.3-P1.90-LS2.4-BR, F.Cu at (278.6, 114.3)
- added K_SW61: DRV5055A4QDBZR, easyeda2kicad:SOT-23-3_L2.9-W1.3-P1.90-LS2.4-BR, F.Cu at (302.4, 114.3)
- added K_SW7: DRV5055A4QDBZR, easyeda2kicad:SOT-23-3_L2.9-W1.3-P1.90-LS2.4-BR, F.Cu at (152.4, 38.1)
- added K_SW8: DRV5055A4QDBZR, easyeda2kicad:SOT-23-3_L2.9-W1.3-P1.90-LS2.4-BR, F.Cu at (171.4, 38.1)
- added K_SW9: DRV5055A4QDBZR, easyeda2kicad:SOT-23-3_L2.9-W1.3-P1.90-LS2.4-BR, F.Cu at (190.5, 38.1)
- added _SW1: RESET, easyeda2kicad:SW-SMD_4P-L5.1-W5.1-P3.70-LS6.5-TL_H1.5, F.Cu at (368.5, 211.6)
- added _SW2: BOOTSEL, easyeda2kicad:SW-SMD_4P-L5.1-W5.1-P3.70-LS6.5-TL_H1.5, F.Cu at (368.5, 217.9)
- C12, C13: value 100nF -> 33pF
- C14, C15, C18, C33, C34, C35, C37, C39, C40, C41, C43, C45, C47, C49, C53: value 100nF -> 1uF
- C17, C20: value 1uF -> 10uF; footprint Capacitor_SMD:C_0603_1608Metric_Pad1.08x0.95mm_HandSolder -> Capacitor_SMD:C_1206_3216Metric_Pad1.33x1.80mm_HandSolder
- C2: value 100nF -> 22uF; footprint Capacitor_SMD:C_0603_1608Metric_Pad1.08x0.95mm_HandSolder -> Capacitor_SMD:C_1206_3216Metric_Pad1.33x1.80mm_HandSolder
- C21, C32: value 1uF -> 100nF
- C22: value 100nF -> 4.7nF
- C24, C25: value 100nF -> 1nF
- C29: value 100nF -> 10uF; footprint Capacitor_SMD:C_0603_1608Metric_Pad1.08x0.95mm_HandSolder -> Capacitor_SMD:C_1206_3216Metric_Pad1.33x1.80mm_HandSolder
- C30: value 100nF -> 10nF
- R1, R3: value 0 -> 22
- R10, R15, R16, R2, R35, R37, R38, R55, R57, R58, R75, R77, R78: value 0 -> 10k
- R11, R4: value 0 -> 5.1k
- R12, R14: value 0 -> 10k 0.1%
- R13: value 0 -> 10
- R19, R20, R25, R30, R31, R45, R50, R51, R65, R70, R71, R85, R90, R91: value 10k -> 0
- R5, R8: value 0 -> 100k
- R6, R7: value 0 -> 1k
- R9: value 0 -> 1M
- U1: value RP2040 -> RT9013-33GB; footprint easyeda2kicad:LQFN-56_L7.0-W7.0-P0.4-EP -> easyeda2kicad:SOT-23-5_L3.0-W1.7-P0.95-LS2.8-BL
- U2: value ADS7953QDBTRQ1 -> W25Q128JVSIQTR; footprint easyeda2kicad:TSSOP-38_L9.7-W4.4-P0.50-LS6.4-BL -> easyeda2kicad:SOIC-8_L5.3-W5.3-P1.27-LS8.0-BL
- U3: value ADS7953QDBTRQ1 -> RP2040; footprint easyeda2kicad:TSSOP-38_L9.7-W4.4-P0.50-LS6.4-BL -> easyeda2kicad:LQFN-56_L7.0-W7.0-P0.4-EP
- U4: value ADS7953QDBTRQ1 -> OPA320AIDBVR; footprint easyeda2kicad:TSSOP-38_L9.7-W4.4-P0.50-LS6.4-BL -> easyeda2kicad:SOT-23-5_L3.0-W1.7-P0.95-LS2.8-BR
- U7: value W25Q128JVSIQTR -> ADS7953QDBTRQ1; footprint easyeda2kicad:SOIC-8_L5.3-W5.3-P1.27-LS8.0-BL -> easyeda2kicad:TSSOP-38_L9.7-W4.4-P0.50-LS6.4-BL
- U8: value RT9013-33GB -> ADS7953QDBTRQ1; footprint easyeda2kicad:SOT-23-5_L3.0-W1.7-P0.95-LS2.8-BL -> easyeda2kicad:TSSOP-38_L9.7-W4.4-P0.50-LS6.4-BL
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Connections:
- C1 pad 2: Net-(SW1-VCC) -> GND
- C10 pad 1: +5VA -> +3V3
- C10 pad 2: Net-(SW10-VCC) -> GND
- C11 pad 1: +5VA -> +3V3
- C11 pad 2: Net-(SW11-VCC) -> GND
- C12 pad 1: +5VA -> GND
- C12 pad 2: Net-(SW12-VCC) -> /XOUT
- C13 pad 1: +5VA -> /XIN
- C13 pad 2: Net-(SW13-VCC) -> GND
- C14 pad 1: +5VA -> +1V1
- C14 pad 2: Net-(SW14-VCC) -> GND
- C15 pad 1: +5VA -> +3V3
- C15 pad 2: Net-(SW15-VCC) -> GND
- C16 pad 1: +5VA -> /V_Fused
- C16 pad 2: Net-(SW16-VCC) -> GND
- C17 pad 1: +3V3 -> /V_Fused
- C18 pad 1: +5VA -> GND
- C18 pad 2: Net-(SW17-VCC) -> +3V3
- C19 pad 1: +2V5_REF -> +3V3
- C2 pad 2: Net-(SW2-VCC) -> GND
- C20 pad 1: +5VA -> +3V3
- C21 pad 2: +5VA -> +3V3
- C22 pad 1: +5VA -> Net-(C22-Pad1)
- C22 pad 2: Net-(SW18-VCC) -> GND
- C23 pad 1: +5VA -> /RUN
- C23 pad 2: Net-(SW19-VCC) -> GND
- C24 pad 1: +5VA -> GND
- C24 pad 2: Net-(SW20-VCC) -> /GPIO26
- C25 pad 1: +2V5_REF -> /GPIO27
- C27 pad 1: +5VA -> GND
- C27 pad 2: Net-(SW21-VCC) -> +5VA
- C28 pad 1: +5VA -> GND
- C28 pad 2: Net-(SW22-VCC) -> +2V5_REF
- C29 pad 1: +5VA -> +2V5_REF
- C29 pad 2: Net-(SW23-VCC) -> GND
- C3 pad 1: +5VA -> +1V1
- C3 pad 2: Net-(SW3-VCC) -> GND
- C30 pad 1: +5VA -> Net-(U4-IN+)
- C30 pad 2: Net-(SW24-VCC) -> GND
- C31 pad 1: +3V3 -> GND
- C31 pad 2: GND -> +2V5_REF
- C32 pad 1: GND -> +2V5_REF
- C32 pad 2: +5VA -> GND
- C33 pad 1: +5VA -> +3V3
- C33 pad 2: Net-(SW25-VCC) -> GND
- C34 pad 2: Net-(SW26-VCC) -> GND
- C35 pad 1: +5VA -> GND
- C35 pad 2: Net-(SW27-VCC) -> +5VA
- C36 pad 1: +5VA -> GND
- C36 pad 2: Net-(SW28-VCC) -> +5VA
- C37 pad 1: +5VA -> GND
- C37 pad 2: Net-(SW29-VCC) -> +2V5_REF
- C38 pad 1: +5VA -> +2V5_REF
- C38 pad 2: Net-(SW30-VCC) -> GND
- C39 pad 1: +5VA -> +3V3
- C39 pad 2: Net-(SW31-VCC) -> GND
- C4 pad 1: +5VA -> +1V1
- C4 pad 2: Net-(SW4-VCC) -> GND
- C40 pad 2: Net-(SW32-VCC) -> GND
- C41 pad 1: +5VA -> GND
- C41 pad 2: Net-(SW33-VCC) -> +5VA
- C42 pad 1: +5VA -> GND
- C42 pad 2: Net-(SW34-VCC) -> +5VA
- C43 pad 1: +5VA -> GND
- C43 pad 2: Net-(SW35-VCC) -> +2V5_REF
- C44 pad 1: +5VA -> +2V5_REF
- C44 pad 2: Net-(SW36-VCC) -> GND
- C45 pad 1: +2V5_REF -> +3V3
- C47 pad 1: +5VA -> GND
- C47 pad 2: Net-(SW37-VCC) -> +5VA
- C48 pad 1: +5VA -> GND
- C48 pad 2: Net-(SW38-VCC) -> +5VA
- C49 pad 1: +5VA -> GND
- C49 pad 2: Net-(SW39-VCC) -> +2V5_REF
- C5 pad 1: +5VA -> +3V3
- C5 pad 2: Net-(SW5-VCC) -> GND
- C50 pad 1: +5VA -> +2V5_REF
- C50 pad 2: Net-(SW40-VCC) -> GND
- C52 pad 1: GND -> +5VA
- C52 pad 2: +5VA -> GND
- C53 pad 1: +5VA -> GND
- C53 pad 2: Net-(SW41-VCC) -> +5VA
- C6 pad 1: +5VA -> +3V3
- C6 pad 2: Net-(SW6-VCC) -> GND
- C7 pad 1: +5VA -> +3V3
- C7 pad 2: Net-(SW7-VCC) -> GND
- C8 pad 1: +5VA -> +3V3
- C8 pad 2: Net-(SW8-VCC) -> GND
- C9 pad 1: +5VA -> +3V3
- C9 pad 2: Net-(SW9-VCC) -> GND
- R1 pad 1: Net-(U2-CH0) -> /USB_DP
- R1 pad 2: /ADC1/KEY_1_0 -> Net-(U3-USB_DP)
- R10 pad 1: Net-(U2-CH9) -> +3V3
- R10 pad 2: /ADC1/KEY_1_9 -> /RUN
- R11 pad 1: Net-(U2-CH10) -> Net-(USBC1-CC2)
- R11 pad 2: /ADC1/KEY_1_10 -> GND
- R12 pad 1: Net-(U2-CH11) -> +5VA
- R12 pad 2: /ADC1/KEY_1_11 -> Net-(U4-IN+)
- R13 pad 1: Net-(U2-CH12) -> Net-(U4-IN-)
- R13 pad 2: /ADC1/KEY_1_12 -> +2V5_REF
- R14 pad 1: Net-(U2-CH13) -> Net-(U4-IN+)
- R14 pad 2: /ADC1/KEY_1_13 -> GND
- R15 pad 1: Net-(U2-CH14) -> Net-(U5-GPIO3)
- R15 pad 2: /ADC1/KEY_1_14 -> +3V3
- R16 pad 1: Net-(U2-CH15) -> Net-(U5-GPIO2)
- R16 pad 2: /ADC1/KEY_1_15 -> +3V3
- R17 pad 1: Net-(U2-GPIO2) -> Net-(U5-GPIO1)
- R17 pad 2: +3V3 -> GND
- R18 pad 1: Net-(U2-GPIO3) -> Net-(U5-GPIO0)
- R18 pad 2: +3V3 -> GND
- R19 pad 1: Net-(U2-GPIO1) -> Net-(U5-CH15)
- R19 pad 2: GND -> /ADC1/CH15
- R2 pad 1: Net-(U2-CH1) -> +3V3
- R2 pad 2: /ADC1/KEY_1_1 -> /FLASH_~{CS}
- R20 pad 1: Net-(U2-GPIO0) -> Net-(U5-CH0)
- R20 pad 2: GND -> /ADC1/CH0
- R21 pad 1: Net-(U3-CH15) -> Net-(U5-CH14)
- R21 pad 2: /ADC2/KEY_1_15 -> /ADC1/CH14
- R22 pad 1: Net-(U3-CH13) -> Net-(U5-CH1)
- R22 pad 2: /ADC2/KEY_1_13 -> /ADC1/CH1
- R23 pad 1: Net-(U3-CH11) -> Net-(U5-CH13)
- R23 pad 2: /ADC2/KEY_1_11 -> /ADC1/CH13
- R24 pad 1: Net-(U3-CH9) -> Net-(U5-CH2)
- R24 pad 2: /ADC2/KEY_1_9 -> /ADC1/CH2
- R25 pad 1: Net-(U3-GPIO3) -> Net-(U5-CH12)
- R25 pad 2: +3V3 -> /ADC1/CH12
- R26 pad 1: Net-(U3-CH14) -> Net-(U5-CH3)
- R26 pad 2: /ADC2/KEY_1_14 -> /ADC1/CH3
- R27 pad 1: Net-(U3-CH12) -> Net-(U5-CH11)
- R27 pad 2: /ADC2/KEY_1_12 -> /ADC1/CH11
- R28 pad 1: Net-(U3-CH10) -> Net-(U5-CH4)
- R28 pad 2: /ADC2/KEY_1_10 -> /ADC1/CH4
- R29 pad 1: Net-(U3-CH8) -> Net-(U5-CH10)
- R29 pad 2: /ADC2/KEY_1_8 -> /ADC1/CH10
- R3 pad 1: Net-(U2-CH2) -> /USB_DN
- R3 pad 2: /ADC1/KEY_1_2 -> Net-(U3-USB_DM)
- R30 pad 1: Net-(U3-GPIO2) -> Net-(U5-CH5)
- R30 pad 2: +3V3 -> /ADC1/CH5
- R31 pad 1: Net-(U3-GPIO1) -> Net-(U5-CH9)
- R31 pad 2: GND -> /ADC1/CH9
- R32 pad 1: Net-(U3-CH0) -> Net-(U5-CH6)
- R32 pad 2: /ADC2/KEY_1_0 -> /ADC1/CH6
- R33 pad 1: Net-(U3-CH2) -> Net-(U5-CH8)
- R33 pad 2: /ADC2/KEY_1_2 -> /ADC1/CH8
- R34 pad 1: Net-(U3-CH4) -> Net-(U5-CH7)
- R34 pad 2: /ADC2/KEY_1_4 -> /ADC1/CH7
- R35 pad 1: Net-(U3-CH6) -> Net-(U6-GPIO3)
- R35 pad 2: /ADC2/KEY_1_6 -> +3V3
- R36 pad 1: Net-(U3-GPIO0) -> Net-(U6-GPIO2)
- R36 pad 2: GND -> +3V3
- R37 pad 1: Net-(U3-CH1) -> Net-(U6-GPIO1)
- R37 pad 2: /ADC2/KEY_1_1 -> GND
- R38 pad 1: Net-(U3-CH3) -> Net-(U6-GPIO0)
- R38 pad 2: /ADC2/KEY_1_3 -> GND
- R39 pad 1: Net-(U3-CH5) -> Net-(U6-CH15)
- R39 pad 2: /ADC2/KEY_1_5 -> /ADC2/CH15
- R4 pad 1: Net-(U2-CH3) -> Net-(USBC1-CC1)
- R4 pad 2: /ADC1/KEY_1_3 -> GND
- R40 pad 1: Net-(U3-CH7) -> Net-(U6-CH0)
- R40 pad 2: /ADC2/KEY_1_7 -> /ADC2/CH0
- R41 pad 1: Net-(U4-CH15) -> Net-(U6-CH14)
- R41 pad 2: /ADC3/KEY_1_15 -> /ADC2/CH14
- R42 pad 1: Net-(U4-CH13) -> Net-(U6-CH1)
- R42 pad 2: /ADC3/KEY_1_13 -> /ADC2/CH1
- R43 pad 1: Net-(U4-CH11) -> Net-(U6-CH13)
- R43 pad 2: /ADC3/KEY_1_11 -> /ADC2/CH13
- R44 pad 1: Net-(U4-CH9) -> Net-(U6-CH2)
- R44 pad 2: /ADC3/KEY_1_9 -> /ADC2/CH2
- R45 pad 1: Net-(U4-GPIO3) -> Net-(U6-CH12)
- R45 pad 2: +3V3 -> /ADC2/CH12
- R46 pad 1: Net-(U4-CH14) -> Net-(U6-CH3)
- R46 pad 2: /ADC3/KEY_1_14 -> /ADC2/CH3
- R47 pad 1: Net-(U4-CH12) -> Net-(U6-CH11)
- R47 pad 2: /ADC3/KEY_1_12 -> /ADC2/CH11
- R48 pad 1: Net-(U4-CH10) -> Net-(U6-CH4)
- R48 pad 2: /ADC3/KEY_1_10 -> /ADC2/CH4
- R49 pad 1: Net-(U4-CH8) -> Net-(U6-CH10)
- R49 pad 2: /ADC3/KEY_1_8 -> /ADC2/CH10
- R5 pad 1: Net-(U2-CH4) -> /GPIO26
- R5 pad 2: /ADC1/KEY_1_4 -> Net-(USBC1-CC1)
- R50 pad 1: Net-(U4-GPIO2) -> Net-(U6-CH5)
- R50 pad 2: +3V3 -> /ADC2/CH5
- R51 pad 1: Net-(U4-GPIO1) -> Net-(U6-CH9)
- R51 pad 2: GND -> /ADC2/CH9
- R52 pad 1: Net-(U4-CH0) -> Net-(U6-CH6)
- R52 pad 2: /ADC3/KEY_1_0 -> /ADC2/CH6
- R53 pad 1: Net-(U4-CH2) -> Net-(U6-CH8)
- R53 pad 2: /ADC3/KEY_1_2 -> /ADC2/CH8
- R54 pad 1: Net-(U4-CH4) -> Net-(U6-CH7)
- R54 pad 2: /ADC3/KEY_1_4 -> /ADC2/CH7
- R55 pad 1: Net-(U4-CH6) -> Net-(U7-GPIO3)
- R55 pad 2: /ADC3/KEY_1_6 -> +3V3
- R56 pad 1: Net-(U4-GPIO0) -> Net-(U7-GPIO2)
- R56 pad 2: GND -> +3V3
- R57 pad 1: Net-(U4-CH1) -> Net-(U7-GPIO1)
- R57 pad 2: /ADC3/KEY_1_1 -> GND
- R58 pad 1: Net-(U4-CH3) -> Net-(U7-GPIO0)
- R58 pad 2: /ADC3/KEY_1_3 -> GND
- R59 pad 1: Net-(U4-CH5) -> Net-(U7-CH15)
- R59 pad 2: /ADC3/KEY_1_5 -> /ADC3/CH15
- R6 pad 1: Net-(U2-CH5) -> /XIN
- R6 pad 2: /ADC1/KEY_1_5 -> Net-(U3-XOUT)
- R60 pad 1: Net-(U4-CH7) -> Net-(U7-CH0)
- R60 pad 2: /ADC3/KEY_1_7 -> /ADC3/CH0
- R61 pad 1: Net-(U5-CH15) -> Net-(U7-CH14)
- R61 pad 2: /ADC4/KEY_1_15 -> /ADC3/CH14
- R62 pad 1: Net-(U5-CH13) -> Net-(U7-CH1)
- R62 pad 2: /ADC4/KEY_1_13 -> /ADC3/CH1
- R63 pad 1: Net-(U5-CH11) -> Net-(U7-CH13)
- R63 pad 2: /ADC4/KEY_1_11 -> /ADC3/CH13
- R64 pad 1: Net-(U5-CH9) -> Net-(U7-CH2)
- R64 pad 2: /ADC4/KEY_1_9 -> /ADC3/CH2
- R65 pad 1: Net-(U5-GPIO3) -> Net-(U7-CH12)
- R65 pad 2: +3V3 -> /ADC3/CH12
- R66 pad 1: Net-(U5-CH14) -> Net-(U7-CH3)
- R66 pad 2: /ADC4/KEY_1_14 -> /ADC3/CH3
- R67 pad 1: Net-(U5-CH12) -> Net-(U7-CH11)
- R67 pad 2: /ADC4/KEY_1_12 -> /ADC3/CH11
- R68 pad 1: Net-(U5-CH10) -> Net-(U7-CH4)
- R68 pad 2: /ADC4/KEY_1_10 -> /ADC3/CH4
- R69 pad 1: Net-(U5-CH8) -> Net-(U7-CH10)
- R69 pad 2: /ADC4/KEY_1_8 -> /ADC3/CH10
- R7 pad 1: Net-(U2-CH6) -> /FLASH_~{CS}
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
Commit message: PCB rough placements
Parts:
- removed R31, R32, R33, R34, R39, R40, R41, R42, R43, R44, R45, R46, R47, R48, R49, R50, R51, R52, R53, R54, R59, R60, R61, R62, R63, R64, R65, R66, R67, R68, R69, R70, R71, R72, R73, R74, R79, R80, R81, R82, R83, R84, R85, R86, R87, R88, R89, R90, R91, R92, R93, R94: 0, Resistor_SMD:R_0603_1608Metric_Pad0.98x0.95mm_HandSolder
- removed R35, R36, R37, R38, R55, R56, R57, R58, R75, R76, R77, R78: 10k, Resistor_SMD:R_0603_1608Metric_Pad0.98x0.95mm_HandSolder
- C1, C10, C11, C12, C13, C14, C15, C16, C17, C18, C19, C2, C20, C21, C22, C23, C24, C25, C26, C27, C28, C29, C3, C30, C31, C32, C33, C34, C35, C36, C37, C38, C39, C4, C40, C41, C42, C43, C44, C45, C46, C47, C48, C49, C5, C50, C51, C52, C53, C6, C7, C8, C9, D1, D2, F1, FB1, R1, R10, R11, R12, R13, R14, R15, R16, R17, R18, R2, R3, R4, R5, R6, R7, R8, R9, SW1, SW2, SW3, U1, U2, U3, U4, U5, U6, U7, U8, USBC1, X1, _SW1, _SW2: moved to B.Cu
- R19, R20, R21, R22, R23, R24, R25, R26, R27, R28, R29, R30: value 0 -> 10k; moved to B.Cu
- moved U6 368.0 mm to (53.0, 55.0), turned to 90 degrees
- moved U5 345.9 mm to (47.9, 37.5), turned to -90 degrees
- moved U7 330.9 mm to (56.0, 74.0), turned to 90 degrees
- moved U8 289.7 mm to (64.0, 92.0), turned to 90 degrees
- moved USBC1 263.1 mm to (181.0, 29.0)
- moved FB1 194.9 mm to (186.0, 170.0), turned to 180 degrees
- moved U1 194.9 mm to (186.0, 166.4), turned to 180 degrees
- moved U2 194.5 mm to (186.2, 176.7), turned to 180 degrees
- moved SW1 194.5 mm to (191.7, 198.5), turned to 180 degrees
- moved D1 193.0 mm to (187.0, 183.5), turned to 180 degrees
- moved _SW1 187.5 mm to (189.9, 154.7), turned to 180 degrees
- moved _SW2 187.5 mm to (189.9, 161.0), turned to 180 degrees
- moved X1 185.3 mm to (191.1, 166.5), turned to 180 degrees
- moved U3 179.6 mm to (194.0, 176.0), turned to 180 degrees
- moved C36 179.1 mm to (195.8, 188.6), turned to 180 degrees
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Connections:
- R19 pad 1: Net-(U5-CH15) -> Net-(U6-GPIO3)
- R19 pad 2: /ADC1/CH15 -> +3V3
- R20 pad 1: Net-(U5-CH0) -> Net-(U6-GPIO2)
- R20 pad 2: /ADC1/CH0 -> +3V3
- R21 pad 1: Net-(U5-CH14) -> Net-(U6-GPIO1)
- R21 pad 2: /ADC1/CH14 -> GND
- R22 pad 1: Net-(U5-CH1) -> Net-(U6-GPIO0)
- R22 pad 2: /ADC1/CH1 -> GND
- R23 pad 1: Net-(U5-CH13) -> Net-(U7-GPIO3)
- R23 pad 2: /ADC1/CH13 -> +3V3
- R24 pad 1: Net-(U5-CH2) -> Net-(U7-GPIO2)
- R24 pad 2: /ADC1/CH2 -> +3V3
- R25 pad 1: Net-(U5-CH12) -> Net-(U7-GPIO1)
- R25 pad 2: /ADC1/CH12 -> GND
- R26 pad 1: Net-(U5-CH3) -> Net-(U7-GPIO0)
- R26 pad 2: /ADC1/CH3 -> GND
- R27 pad 1: Net-(U5-CH11) -> Net-(U8-GPIO3)
- R27 pad 2: /ADC1/CH11 -> +3V3
- R28 pad 1: Net-(U5-CH4) -> Net-(U8-GPIO2)
- R28 pad 2: /ADC1/CH4 -> +3V3
- R29 pad 1: Net-(U5-CH10) -> Net-(U8-GPIO1)
- R29 pad 2: /ADC1/CH10 -> GND
- R30 pad 1: Net-(U5-CH5) -> Net-(U8-GPIO0)
- R30 pad 2: /ADC1/CH5 -> GND
- U5 pad 11: Net-(U5-CH15) -> /ADC1/CH15
- U5 pad 12: Net-(U5-CH14) -> /ADC1/CH14
- U5 pad 13: Net-(U5-CH13) -> /ADC1/CH13
- U5 pad 14: Net-(U5-CH12) -> /ADC1/CH12
- U5 pad 15: Net-(U5-CH11) -> /ADC1/CH11
- U5 pad 16: Net-(U5-CH10) -> /ADC1/CH10
- U5 pad 17: Net-(U5-CH9) -> /ADC1/CH9
- U5 pad 18: Net-(U5-CH8) -> /ADC1/CH8
- U5 pad 21: Net-(U5-CH7) -> /ADC1/CH7
- U5 pad 22: Net-(U5-CH6) -> /ADC1/CH6
- U5 pad 23: Net-(U5-CH5) -> /ADC1/CH5
- U5 pad 24: Net-(U5-CH4) -> /ADC1/CH4
- U5 pad 25: Net-(U5-CH3) -> /ADC1/CH3
- U5 pad 26: Net-(U5-CH2) -> /ADC1/CH2
- U5 pad 27: Net-(U5-CH1) -> /ADC1/CH1
- U5 pad 28: Net-(U5-CH0) -> /ADC1/CH0
- U6 pad 11: Net-(U6-CH15) -> /ADC2/CH15
- U6 pad 12: Net-(U6-CH14) -> /ADC2/CH14
- U6 pad 13: Net-(U6-CH13) -> /ADC2/CH13
- U6 pad 14: Net-(U6-CH12) -> /ADC2/CH12
- U6 pad 15: Net-(U6-CH11) -> /ADC2/CH11
- U6 pad 16: Net-(U6-CH10) -> /ADC2/CH10
- U6 pad 17: Net-(U6-CH9) -> /ADC2/CH9
- U6 pad 18: Net-(U6-CH8) -> /ADC2/CH8
- U6 pad 21: Net-(U6-CH7) -> /ADC2/CH7
- U6 pad 22: Net-(U6-CH6) -> /ADC2/CH6
- U6 pad 23: Net-(U6-CH5) -> /ADC2/CH5
- U6 pad 24: Net-(U6-CH4) -> /ADC2/CH4
- U6 pad 25: Net-(U6-CH3) -> /ADC2/CH3
- U6 pad 26: Net-(U6-CH2) -> /ADC2/CH2
- U6 pad 27: Net-(U6-CH1) -> /ADC2/CH1
- U6 pad 28: Net-(U6-CH0) -> /ADC2/CH0
- U7 pad 11: Net-(U7-CH15) -> /ADC3/CH15
- U7 pad 12: Net-(U7-CH14) -> /ADC3/CH14
- U7 pad 13: Net-(U7-CH13) -> /ADC3/CH13
- U7 pad 14: Net-(U7-CH12) -> /ADC3/CH12
- U7 pad 15: Net-(U7-CH11) -> /ADC3/CH11
- U7 pad 16: Net-(U7-CH10) -> /ADC3/CH10
- U7 pad 17: Net-(U7-CH9) -> /ADC3/CH9
- U7 pad 18: Net-(U7-CH8) -> /ADC3/CH8
- U7 pad 21: Net-(U7-CH7) -> /ADC3/CH7
- U7 pad 22: Net-(U7-CH6) -> /ADC3/CH6
- U7 pad 23: Net-(U7-CH5) -> /ADC3/CH5
- U7 pad 24: Net-(U7-CH4) -> /ADC3/CH4
- U7 pad 25: Net-(U7-CH3) -> /ADC3/CH3
- U7 pad 26: Net-(U7-CH2) -> /ADC3/CH2
- U7 pad 27: Net-(U7-CH1) -> /ADC3/CH1
- U7 pad 28: Net-(U7-CH0) -> /ADC3/CH0
- U8 pad 11: Net-(U8-CH15) -> /ADC4/CH15
- U8 pad 12: Net-(U8-CH14) -> /ADC4/CH14
- U8 pad 13: Net-(U8-CH13) -> /ADC4/CH13
- U8 pad 14: Net-(U8-CH12) -> /ADC4/CH12
- U8 pad 15: Net-(U8-CH11) -> /ADC4/CH11
- U8 pad 16: Net-(U8-CH10) -> /ADC4/CH10
- U8 pad 17: Net-(U8-CH9) -> /ADC4/CH9
- U8 pad 18: Net-(U8-CH8) -> /ADC4/CH8
- U8 pad 21: Net-(U8-CH7) -> /ADC4/CH7
- U8 pad 22: Net-(U8-CH6) -> /ADC4/CH6
- U8 pad 23: Net-(U8-CH5) -> /ADC4/CH5
- U8 pad 24: Net-(U8-CH4) -> /ADC4/CH4
- U8 pad 25: Net-(U8-CH3) -> /ADC4/CH3
- U8 pad 26: Net-(U8-CH2) -> /ADC4/CH2
- U8 pad 27: Net-(U8-CH1) -> /ADC4/CH1
- U8 pad 28: Net-(U8-CH0) -> /ADC4/CH0
Other:
- board outline added: 285 x 100 mm

Commit message: PCB layout v1
Parts:
- removed C51, C52, C53: 1uF, Capacitor_SMD:C_0603_1608Metric_Pad1.08x0.95mm_HandSolder
- removed SW1, SW2, SW3: DRV5055A4QDBZR, easyeda2kicad:SOT-23-3_L2.9-W1.3-P1.90-LS2.4-BR
- C36, C38, C44, C48, C50: value 100nF -> 1uF
- C37, C47: value 1uF -> 100nF
- R7, _SW1, _SW2: moved to F.Cu
- moved U5 208.1 mm to (255.8, 47.0)
- moved U8 202.4 mm to (265.5, 110.9), turned to -90 degrees
- moved U6 199.8 mm to (252.3, 69.9), turned to -90 degrees
- moved U7 188.5 mm to (243.8, 90.1), turned to -90 degrees
- moved R18 185.4 mm to (254.5, 39.8), turned to 90 degrees
- moved R16 182.7 mm to (259.0, 39.8), turned to 90 degrees
- moved R17 182.5 mm to (253.0, 39.8), turned to 90 degrees
- moved R15 179.8 mm to (257.5, 39.8), turned to 90 degrees
- moved C34 172.7 mm to (261.8, 45.0), turned to 0 degrees
- moved C32 170.0 mm to (260.8, 42.5), turned to 90 degrees
- moved U4 168.7 mm to (282.8, 31.5), turned to 0 degrees
- moved C29 168.7 mm to (274.2, 31.0), turned to 90 degrees
- moved C31 168.5 mm to (262.2, 42.5), turned to -90 degrees
- moved C35 168.1 mm to (249.9, 46.6), turned to 0 degrees
- moved R14 166.7 mm to (285.8, 29.8), turned to 90 degrees
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Connections:
- net Net-(U3-USB_DM) renamed /RP_USB_DN
- net Net-(U3-USB_DP) renamed /RP_USB_DP
- C36 pad 2: +5VA -> +2V5_REF
- C37 pad 1: GND -> +2V5_REF
- C37 pad 2: +2V5_REF -> GND
- C38 pad 1: +2V5_REF -> +3V3
- C39 pad 1: +3V3 -> +5VA
- C40 pad 1: +5VA -> GND
- C40 pad 2: GND -> +5VA
- C41 pad 2: +5VA -> +2V5_REF
- C42 pad 1: GND -> +2V5_REF
- C42 pad 2: +5VA -> GND
- C43 pad 1: GND -> +3V3
- C43 pad 2: +2V5_REF -> GND
- C44 pad 1: +2V5_REF -> +5VA
- C45 pad 1: +3V3 -> GND
- C45 pad 2: GND -> +5VA
- C46 pad 1: +5VA -> GND
- C46 pad 2: GND -> +2V5_REF
- C47 pad 1: GND -> +2V5_REF
- C47 pad 2: +5VA -> GND
- C48 pad 1: GND -> +3V3
- C48 pad 2: +5VA -> GND
- C49 pad 1: GND -> +5VA
- C49 pad 2: +2V5_REF -> GND
- C50 pad 1: +2V5_REF -> GND
- C50 pad 2: GND -> +5VA
- K_SW17 pad 2: /ADC2/CH1 -> /ADC2/CH0
- K_SW18 pad 2: /ADC2/CH2 -> /ADC2/CH1
- K_SW19 pad 2: /ADC2/CH3 -> /ADC2/CH2
- K_SW20 pad 2: /ADC2/CH4 -> /ADC2/CH3
- K_SW21 pad 2: /ADC2/CH5 -> /ADC2/CH4
- K_SW22 pad 2: /ADC2/CH6 -> /ADC2/CH5
- K_SW23 pad 2: /ADC2/CH7 -> /ADC2/CH6
- K_SW24 pad 2: /ADC2/CH8 -> /ADC2/CH7
- K_SW25 pad 2: /ADC2/CH9 -> /ADC2/CH8
- K_SW26 pad 2: /ADC2/CH10 -> /ADC2/CH9
- K_SW27 pad 2: /ADC2/CH11 -> /ADC2/CH10
- K_SW28 pad 2: /ADC2/CH12 -> /ADC2/CH11
- K_SW29 pad 2: /ADC2/CH13 -> /ADC2/CH12
- K_SW30 pad 2: /ADC2/CH14 -> /ADC2/CH13
- K_SW31 pad 2: /ADC2/CH15 -> /ADC2/CH14
- K_SW32 pad 2: /ADC3/CH1 -> /ADC2/CH15
- K_SW33 pad 2: /ADC3/CH2 -> /ADC3/CH0
- K_SW34 pad 2: /ADC3/CH3 -> /ADC3/CH1
- K_SW35 pad 2: /ADC3/CH4 -> /ADC3/CH2
- K_SW36 pad 2: /ADC3/CH5 -> /ADC3/CH3
- K_SW37 pad 2: /ADC3/CH6 -> /ADC3/CH4
- K_SW38 pad 2: /ADC3/CH7 -> /ADC3/CH5
- K_SW39 pad 2: /ADC3/CH8 -> /ADC3/CH6
- K_SW40 pad 2: /ADC3/CH9 -> /ADC3/CH7
- K_SW41 pad 2: /ADC3/CH10 -> /ADC3/CH8
- K_SW42 pad 2: /ADC3/CH11 -> /ADC3/CH9
- K_SW43 pad 2: /ADC3/CH12 -> /ADC3/CH10
- K_SW44 pad 2: /ADC3/CH13 -> /ADC3/CH11
- K_SW45 pad 2: /ADC3/CH14 -> /ADC3/CH12
- K_SW46 pad 2: /ADC3/CH15 -> /ADC3/CH13
- K_SW47 pad 2: /ADC4/CH1 -> /ADC3/CH14
- K_SW48 pad 2: /ADC4/CH2 -> /ADC3/CH15
- K_SW49 pad 2: /ADC4/CH3 -> /ADC4/CH0
- K_SW50 pad 2: /ADC4/CH4 -> /ADC4/CH1
- K_SW51 pad 2: /ADC4/CH5 -> /ADC4/CH2
- K_SW52 pad 2: /ADC4/CH6 -> /ADC4/CH3
- K_SW53 pad 2: /ADC4/CH7 -> /ADC4/CH4
- K_SW54 pad 2: /ADC4/CH8 -> /ADC4/CH5
- K_SW55 pad 2: /ADC4/CH9 -> /ADC4/CH6
- K_SW56 pad 2: /ADC4/CH10 -> /ADC4/CH7
- K_SW57 pad 2: /ADC4/CH11 -> /ADC4/CH8
- K_SW58 pad 2: /ADC4/CH12 -> /ADC4/CH9
- K_SW59 pad 2: /ADC4/CH13 -> /ADC4/CH10
- K_SW60 pad 2: /ADC4/CH14 -> /ADC4/CH11
- K_SW61 pad 2: /ADC4/CH15 -> /ADC4/CH12
- R6 pad 1: /XIN -> /XOUT
- U3 pad 11: /GPIO8 -> unconnected-(U3-GPIO8-Pad11)
- U3 pad 12: /GPIO9 -> unconnected-(U3-GPIO9-Pad12)
- U3 pad 13: /GPIO10 -> unconnected-(U3-GPIO10-Pad13)
- U3 pad 14: /GPIO11 -> unconnected-(U3-GPIO11-Pad14)
- U3 pad 15: /GPIO12 -> unconnected-(U3-GPIO12-Pad15)
- U3 pad 16: /GPIO13 -> unconnected-(U3-GPIO13-Pad16)
- U3 pad 17: /GPIO14 -> unconnected-(U3-GPIO14-Pad17)
- U3 pad 18: /GPIO15 -> unconnected-(U3-GPIO15-Pad18)
- U3 pad 2: /GPIO0 -> ADC_MISO
- U3 pad 20: /XOUT -> /XIN
- U3 pad 27: /GPIO16 -> unconnected-(U3-GPIO16-Pad27)
- U3 pad 28: /GPIO17 -> unconnected-(U3-GPIO17-Pad28)
- U3 pad 29: /GPIO18 -> unconnected-(U3-GPIO18-Pad29)
- U3 pad 3: /GPIO1 -> unconnected-(U3-GPIO1-Pad3)
- U3 pad 30: /GPIO19 -> unconnected-(U3-GPIO19-Pad30)
- U3 pad 31: /GPIO20 -> unconnected-(U3-GPIO20-Pad31)
- U3 pad 32: /GPIO21 -> unconnected-(U3-GPIO21-Pad32)
- U3 pad 34: /GPIO22 -> unconnected-(U3-GPIO22-Pad34)
- U3 pad 35: /GPIO23 -> unconnected-(U3-GPIO23-Pad35)
- U3 pad 36: /GPIO24 -> unconnected-(U3-GPIO24-Pad36)
- U3 pad 37: /GPIO25 -> unconnected-(U3-GPIO25-Pad37)
- U3 pad 4: /GPIO2 -> ADC_SCK
- U3 pad 40: /GPIO28 -> unconnected-(U3-GPIO28_ADC2-Pad40)
- U3 pad 41: /GPIO29 -> unconnected-(U3-GPIO29_ADC3-Pad41)
- U3 pad 5: /GPIO3 -> ADC_MOSI
- U3 pad 6: /GPIO4 -> /ADC_~{CS}1
- U3 pad 7: /GPIO5 -> /ADC_~{CS}2
- U3 pad 8: /GPIO6 -> /ADC_~{CS}3
- U3 pad 9: /GPIO7 -> /ADC_~{CS}4
- U5 pad 31: ~{CS} -> /ADC_~{CS}1
- U5 pad 32: SCLK -> ADC_SCK
- U5 pad 33: MOSI -> ADC_MOSI
- U5 pad 34: /GPIO0 -> ADC_MISO
- U6 pad 31: ~{CS} -> /ADC_~{CS}2
- U6 pad 32: SCLK -> ADC_SCK
- U6 pad 33: MOSI -> ADC_MOSI
- U6 pad 34: /GPIO1 -> ADC_MISO
- U7 pad 31: ~{CS} -> /ADC_~{CS}3
- U7 pad 32: SCLK -> ADC_SCK
- U7 pad 33: MOSI -> ADC_MOSI
- U7 pad 34: /GPIO2 -> ADC_MISO
- U8 pad 31: ~{CS} -> /ADC_~{CS}4
- U8 pad 32: SCLK -> ADC_SCK
- U8 pad 33: MOSI -> ADC_MOSI
- U8 pad 34: /GPIO3 -> ADC_MISO
Routing:
- net ADC_MOSI: track 0.00 -> 262.9 mm, vias 0 -> 15
- net ADC_MISO: track 0.00 -> 258.3 mm, vias 0 -> 15
- net ADC_SCK: track 0.00 -> 258.1 mm, vias 0 -> 15
- net /ADC1/CH0: track 0.00 -> 222.6 mm, vias 0 -> 3
- net /ADC1/CH14: track 0.00 -> 221.2 mm, vias 0 -> 3
- net /ADC2/CH12: track 0.00 -> 214.7 mm, vias 0 -> 3
- net /ADC1/CH1: track 0.00 -> 204.2 mm, vias 0 -> 3
- net /ADC1/CH15: track 0.00 -> 198.8 mm, vias 0 -> 3
- net /ADC3/CH9: track 0.00 -> 198.0 mm, vias 0 -> 3
- net /ADC2/CH13: track 0.00 -> 189.1 mm, vias 0 -> 3
- net /ADC1/CH2: track 0.00 -> 185.7 mm, vias 0 -> 3
- net /ADC2/CH0: track 0.00 -> 173.4 mm, vias 0 -> 1
- net /ADC2/CH14: track 0.00 -> 171.0 mm, vias 0 -> 3
- net /ADC3/CH10: track 0.00 -> 168.1 mm, vias 0 -> 3
- net /ADC1/CH3: track 0.00 -> 167.4 mm, vias 0 -> 3
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- added copper zone on B.Cu, net /VBUS
- added copper zone on F.Cu, net /VBUS
- added copper zone on B.Cu, net /V_Fused
- added copper zone on F.Cu, net /V_Fused
- added copper zone on B.Cu, net GND
- added copper zone on F.Cu, net GND

Commit message: PCB layout final v1
Parts:
- added REF**: MountingHole_2.7mm_M2.5, MountingHole:MountingHole_2.7mm_M2.5, F.Cu at (157.5, 75.0)
- added REF**: MountingHole_2.7mm_M2.5, MountingHole:MountingHole_2.7mm_M2.5, F.Cu at (170.0, 122.5)
- added REF**: MountingHole_2.7mm_M2.5, MountingHole:MountingHole_2.7mm_M2.5, F.Cu at (35.0, 30.0)
- added REF**: MountingHole_2.7mm_M2.5, MountingHole:MountingHole_2.7mm_M2.5, F.Cu at (162.5, 30.0)
- added REF**: MountingHole_2.7mm_M2.5, MountingHole:MountingHole_2.7mm_M2.5, F.Cu at (310.0, 120.0)
- added REF**: MountingHole_2.7mm_M2.5, MountingHole:MountingHole_2.7mm_M2.5, F.Cu at (310.0, 30.0)
- added REF**: MountingHole_2.7mm_M2.5, MountingHole:MountingHole_2.7mm_M2.5, F.Cu at (35.0, 120.0)
- moved C50 1.97 mm to (260.0, 108.9)
Routing:
- net +3V3: track 46.0 -> 502.3 mm, vias 0 -> 33
- net GND: track 0.00 -> 301.5 mm, vias 13 -> 179
- net +5VA: track 17.1 -> 256.1 mm, vias 0 -> 75
- net +2V5_REF: track 5.98 -> 244.8 mm, vias 0 -> 8
- net /ADC4/CH5: track 0.00 -> 224.4 mm, vias 0 -> 1
- net /ADC4/CH6: track 0.00 -> 200.2 mm, vias 0 -> 1
- net /ADC4/CH7: track 0.00 -> 175.8 mm, vias 0 -> 1
- net /FLASH_~{CS}: track 24.8 -> 161.4 mm, vias 0 -> 5
- net /RUN: track 4.97 -> 122.2 mm, vias 0 -> 3
- net /ADC4/CH8: track 0.00 -> 110.6 mm, vias 0 -> 3
- net /ADC4/CH0: track 0.00 -> 81.6 mm, vias 0 -> 1
- net /ADC4/CH1: track 0.00 -> 64.2 mm, vias 0 -> 1
- net /ADC4/CH4: track 0.00 -> 45.8 mm, vias 0 -> 3
- net /ADC4/CH2: track 0.00 -> 44.4 mm, vias 0 -> 1
- net /ADC4/CH9: track 0.00 -> 36.9 mm, vias 0 -> 3
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- added copper zone on B.Cu, net +5VA

Commit message: 3d changes and text
Other:
- board text added: "stav-keeb-60 v0"
