File: stav-keeb-65.kicad_pcb (KiCad board)
At the start: 2 copper layers, 285 x 100 mm, 225 parts, among them U1 RT9013-33GB, U2 W25Q128JVSIQTR, U3 RP2040, U4 OPA320AIDBVR, U5 ADS7953QDBTRQ1, U6 ADS7953QDBTRQ1, U7 ADS7953QDBTRQ1, U8 ADS7953QDBTRQ1, X1 X322512MSB4SI

Commit message: progress towards v2
Parts:
- removed REF** (x7): MountingHole_2.7mm_M2.5, MountingHole:MountingHole_2.7mm_M2.5
- added R33: 33, Resistor_SMD:R_0402_1005Metric, B.Cu at (287.5, 83.1)
- added R34: 33, Resistor_SMD:R_0402_1005Metric, B.Cu at (244.8, 53.7)
- added R35: 33, Resistor_SMD:R_0402_1005Metric, B.Cu at (244.8, 71.8)
- added R36: 33, Resistor_SMD:R_0402_1005Metric, B.Cu at (244.6, 92.3)
- added R37: 33, Resistor_SMD:R_0402_1005Metric, B.Cu at (244.7, 112.6)
- added R38: 33, Resistor_SMD:R_0402_1005Metric, B.Cu at (286.4, 83.1)
- added R39: 33, Resistor_SMD:R_0402_1005Metric, B.Cu at (288.6, 83.1)
- added R40: 33, Resistor_SMD:R_0402_1005Metric, B.Cu at (289.7, 83.1)
- added R41: 33, Resistor_SMD:R_0402_1005Metric, B.Cu at (282.0, 83.1)
- added R42: 33, Resistor_SMD:R_0402_1005Metric, B.Cu at (283.1, 83.1)
- added R43: 33, Resistor_SMD:R_0402_1005Metric, B.Cu at (284.2, 83.1)
- added R44: 33, Resistor_SMD:R_0402_1005Metric, B.Cu at (285.2, 83.1)
- added R45: 33, Resistor_SMD:R_0402_1005Metric, B.Cu at (270.8, 76.3)
- added R46: 33, Resistor_SMD:R_0402_1005Metric, B.Cu at (270.8, 77.4)
- added R47: 33, Resistor_SMD:R_0402_1005Metric, B.Cu at (270.8, 78.5)
- added R48: 33, Resistor_SMD:R_0402_1005Metric, B.Cu at (270.8, 79.6)
- R1, R10, R11, R13, R15, R16, R17, R18, R19, R2, R20, R21, R22, R23, R24, R25, R26, R27, R28, R29, R3, R30, R4, R5, R6, R7, R8: footprint Resistor_SMD:R_0603_1608Metric_Pad0.98x0.95mm_HandSolder -> Resistor_SMD:R_0402_1005Metric
- R12, R14: footprint Resistor_SMD:R_0603_1608Metric_Pad0.98x0.95mm_HandSolder -> Resistor_SMD:R_0603_1608Metric
- moved C26 73.1 mm to (231.6, 82.1), turned to -90 degrees
- moved C30 73.1 mm to (227.9, 75.9), turned to 90 degrees
- moved R14 71.7 mm to (230.9, 75.9)
- moved C27 71.0 mm to (233.1, 82.1), turned to 90 degrees
- moved U4 70.9 mm to (230.0, 78.9), turned to 180 degrees
- moved R12 70.0 mm to (229.4, 74.8), turned to -90 degrees
- moved R13 66.0 mm to (231.8, 78.9), turned to 0 degrees
- moved C28 63.0 mm to (233.5, 78.0)
- moved C29 60.4 mm to (235.4, 77.3)
- moved C46 28.9 mm to (243.4, 101.0), turned to 0 degrees
- moved C47 27.2 mm to (243.4, 102.5), turned to 180 degrees
- moved R28 27.0 mm to (241.3, 104.7), turned to 180 degrees
- moved C49 26.4 mm to (245.9, 101.5), turned to 90 degrees
- moved R27 25.5 mm to (241.3, 105.7), turned to 180 degrees
- moved C12 25.2 mm to (278.5, 80.0)
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Connections:
- U3 pad 13: unconnected-(U3-GPIO10-Pad13) -> /ADC_MISO0
- U3 pad 14: unconnected-(U3-GPIO11-Pad14) -> /ADC_MISO1
- U3 pad 15: unconnected-(U3-GPIO12-Pad15) -> /ADC_MISO2
- U3 pad 16: unconnected-(U3-GPIO13-Pad16) -> /ADC_MISO3
- U3 pad 17: unconnected-(U3-GPIO14-Pad17) -> /RP2040_MOSI
- U3 pad 18: unconnected-(U3-GPIO15-Pad18) -> /RP2040_SCK
- U3 pad 2: ADC_MISO -> unconnected-(U3-GPIO0-Pad2)
- U3 pad 27: unconnected-(U3-GPIO16-Pad27) -> /RP2040_CS_N
- U3 pad 4: ADC_SCK -> unconnected-(U3-GPIO2-Pad4)
- U3 pad 5: ADC_MOSI -> unconnected-(U3-GPIO3-Pad5)
- U3 pad 6: /ADC_~{CS}1 -> unconnected-(U3-GPIO4-Pad6)
- U3 pad 7: /ADC_~{CS}2 -> unconnected-(U3-GPIO5-Pad7)
- U3 pad 8: /ADC_~{CS}3 -> unconnected-(U3-GPIO6-Pad8)
- U3 pad 9: /ADC_~{CS}4 -> unconnected-(U3-GPIO7-Pad9)
- U5 pad 31: /ADC_~{CS}1 -> /ADC_SC_N0
- U5 pad 32: ADC_SCK -> /ADC_SCK0
- U5 pad 33: ADC_MOSI -> /ADC_MOSI0
- U5 pad 34: ADC_MISO -> Net-(U5-SDO)
- U6 pad 31: /ADC_~{CS}2 -> /ADC_SC_N1
- U6 pad 32: ADC_SCK -> /ADC_SCK1
- U6 pad 33: ADC_MOSI -> /ADC_MOSI1
- U6 pad 34: ADC_MISO -> Net-(U6-SDO)
- U7 pad 31: /ADC_~{CS}3 -> /ADC_SC_N2
- U7 pad 32: ADC_SCK -> /ADC_SCK2
- U7 pad 33: ADC_MOSI -> /ADC_MOSI2
- U7 pad 34: ADC_MISO -> Net-(U7-SDO)
- U8 pad 31: /ADC_~{CS}4 -> /ADC_SC_N3
- U8 pad 32: ADC_SCK -> /ADC_SCK3
- U8 pad 33: ADC_MOSI -> /ADC_MOSI3
- U8 pad 34: ADC_MISO -> Net-(U8-SDO)
Routing:
- net +3V3: track 502.3 -> 24.5 mm, vias 33 -> 4
- net ADC_MOSI: track 263.3 -> 0.00 mm, vias 15 -> 0
- net ADC_MISO: track 260.3 -> 0.00 mm, vias 15 -> 0
- net ADC_SCK: track 258.9 -> 0.00 mm, vias 15 -> 0
- net GND: track 301.5 -> 56.4 mm, vias 179 -> 56
- net +5VA: track 256.1 -> 37.3 mm, vias 75 -> 14
- net /FLASH_~{CS}: track 161.4 -> 13.5 mm, vias 5 -> 0
- net +2V5_REF: track 244.8 -> 108.8 mm, vias 8 -> 0
- net /ADC_MISO0: track 0.00 -> 129.8 mm, vias 0 -> 2
- net /RUN: track 122.2 -> 8.61 mm, vias 3 -> 2
- net /ADC_~{CS}1: track 111.3 -> 0.00 mm, vias 4 -> 0
- net /ADC_MISO1: track 0.00 -> 107.1 mm, vias 0 -> 2
- net /ADC_~{CS}2: track 99.6 -> 0.00 mm, vias 4 -> 0
- net /ADC_~{CS}4: track 94.7 -> 0.00 mm, vias 4 -> 0
- net /ADC_MISO3: track 0.00 -> 83.9 mm, vias 0 -> 2
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- added copper zone on B.Cu, net +2V5_REF
- added copper zone on B.Cu, net +3V3
- added copper zone on In1.Cu, net +5VA
- added copper zone on In2.Cu, net GND
- added copper zone on B.Cu, net Net-(U4-IN+)
- added copper zone on B.Cu, net Net-(U4-IN-)
- removed copper zone on B.Cu, net +5VA
- removed copper zone on F.Cu, net /V_Fused
- removed copper zone on F.Cu, net GND
Other:
- copper layers 2 -> 4

Commit message: more progress towards v2
Parts:
- C1, C16, C19: footprint Capacitor_SMD:C_0603_1608Metric_Pad1.08x0.95mm_HandSolder -> Capacitor_SMD:C_1206_3216Metric
- C10, C11, C12, C13, C14, C15, C18, C21, C22, C23, C24, C25, C26, C27, C28, C3, C30, C31, C32, C33, C34, C35, C36, C37, C38, C39, C4, C40, C41, C42, C43, C44, C45, C46, C47, C48, C49, C5, C50, C6, C7, C8, C9, K_C1, K_C10, K_C11, K_C12, K_C13, K_C14, K_C15, K_C16, K_C17, K_C18, K_C19, K_C2, K_C20, K_C21, K_C22, K_C23, K_C24, K_C25, K_C26, K_C27, K_C28, K_C29, K_C3, K_C30, K_C31, K_C32, K_C33, K_C34, K_C35, K_C36, K_C37, K_C38, K_C39, K_C4, K_C40, K_C41, K_C42, K_C43, K_C44, K_C45, K_C46, K_C47, K_C48, K_C49, K_C5, K_C50, K_C51, K_C52, K_C53, K_C54, K_C55, K_C56, K_C57, K_C58, K_C59, K_C6, K_C60, K_C61, K_C7, K_C8, K_C9: footprint Capacitor_SMD:C_0603_1608Metric_Pad1.08x0.95mm_HandSolder -> Capacitor_SMD:C_0402_1005Metric
- C17, C2, C20: footprint Capacitor_SMD:C_1206_3216Metric_Pad1.33x1.80mm_HandSolder -> Capacitor_SMD:C_1206_3216Metric
- R9: footprint Resistor_SMD:R_0603_1608Metric_Pad0.98x0.95mm_HandSolder -> Resistor_SMD:R_0402_1005Metric
- moved C10 6.02 mm to (279.3, 67.4)
- moved C3 5.78 mm to (280.3, 67.4)
- moved R7 3.04 mm to (190.5, 113.2), turned to 180 degrees
- moved C4 2.83 mm to (277.9, 77.0), turned to 180 degrees
- moved C6 2.57 mm to (275.5, 74.1), turned to -90 degrees
- moved R9 2.55 mm to (174.9, 30.7)
- moved C11 2.50 mm to (276.6, 67.2), turned to 180 degrees
- moved C22 2.15 mm to (174.9, 26.5)
- moved C15 1.92 mm to (276.6, 68.2), turned to 180 degrees
- moved C2 1.82 mm to (199.6, 35.7), turned to -90 degrees
- moved C18 1.75 mm to (283.4, 57.8)
- moved C21 1.75 mm to (283.4, 59.3)
- moved R2 1.75 mm to (291.2, 59.0)
- moved U2 1.75 mm to (287.7, 62.3)
- moved C14 1.50 mm to (278.1, 67.7)
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Routing:
- net /ADC_MISO0: track 129.8 -> 105.7 mm
- net /ADC_MISO1: track 107.1 -> 85.7 mm
- net Net-(C22-Pad1): track 0.00 -> 20.8 mm
- net /ADC_MISO2: track 82.1 -> 65.3 mm
- net +3V3: track 24.5 -> 11.4 mm, vias 4 -> 0
- net +1V1: track 15.4 -> 3.92 mm, vias 4 -> 0
- net /FLASH_~{CS}: track 13.5 -> 20.3 mm
- net /ADC_MISO3: track 83.9 -> 77.4 mm, vias 2 -> 0
- net /FLASH_SD1: track 12.1 -> 18.2 mm, vias 2 -> 0
- net /ADC1/CH2: track 186.1 -> 191.8 mm
- net /FLASH_SD2: track 11.1 -> 16.5 mm, vias 2 -> 0
- net /ADC1/CH15: track 189.5 -> 194.7 mm
- net /ADC2/CH12: track 213.7 -> 218.1 mm
- net /ADC2/CH14: track 168.0 -> 171.8 mm
- net /ADC1/CH14: track 214.0 -> 217.5 mm
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
Commit message: closer to v2
Parts:
- C22: footprint Capacitor_SMD:C_0402_1005Metric -> Capacitor_SMD:C_1206_3216Metric
- moved C40 6.73 mm to (248.0, 70.8), turned to 0 degrees
- moved C35 5.81 mm to (249.3, 53.8), turned to 0 degrees
- moved C50 5.26 mm to (247.2, 111.6), turned to 0 degrees
- moved C38 3.58 mm to (243.1, 70.7), turned to 0 degrees
- moved C45 3.24 mm to (247.2, 91.5), turned to 0 degrees
- moved C48 2.86 mm to (243.2, 111.8), turned to 0 degrees
- moved C33 1.98 mm to (243.4, 52.8), turned to 0 degrees
- moved C49 1.52 mm to (245.3, 102.9), turned to 0 degrees
- moved C43 1.51 mm to (243.1, 91.5), turned to 0 degrees
- moved C39 1.50 mm to (245.4, 61.6), turned to 0 degrees
- moved C22 1.46 mm to (173.5, 26.9)
- moved R22 1.32 mm to (241.5, 67.8)
- moved R21 1.19 mm to (241.5, 68.8)
- moved C34 0.98 mm to (245.4, 43.6), turned to 0 degrees
- moved C18 0.93 mm to (284.1, 58.4)
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Routing:
- net GND: track 56.8 -> 453.8 mm, vias 51 -> 282
- net +5VA: track 37.2 -> 182.2 mm, vias 14 -> 112
- net /FLASH_~{CS}: track 20.3 -> 156.0 mm, vias 0 -> 3
- net /RUN: track 8.61 -> 144.2 mm, vias 2 -> 6
- net +3V3: track 11.4 -> 30.3 mm, vias 0 -> 23
- net +1V1: track 3.92 -> 16.8 mm, vias 0 -> 2
- net Net-(_SW2-A): track 0.00 -> 7.01 mm
- net /ADC1/CH1: track 207.7 -> 213.1 mm
- net /ADC1/CH0: track 224.8 -> 230.0 mm
- net Net-(C22-Pad1): track 20.8 -> 25.5 mm
- net /ADC2/CH1: track 157.0 -> 161.3 mm
- net /ADC2/CH0: track 175.6 -> 179.4 mm
- net /ADC3/CH0: track 135.9 -> 132.6 mm
- net /XOUT: track 0.00 -> 2.46 mm
- net /ADC_MOSI3: track 63.2 -> 65.6 mm
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- added copper zone on B.Cu, net +5VA

Commit message: version v2a
Parts:
- moved C23 0.75 mm to (273.5, 80.3), turned to 180 degrees
- moved R10 0.66 mm to (273.5, 79.3), turned to 0 degrees
Routing:
- net +3V3: track 30.3 -> 441.4 mm, vias 23 -> 30
- net GND: track 453.8 -> 440.7 mm, vias 282 -> 278
- net +5VA: track 182.2 -> 178.2 mm
- net /RUN: track 144.2 -> 141.0 mm, vias 6 -> 7
- net /ADC4/CH7: track 166.1 -> 164.0 mm
- net Net-(C22-Pad1): track 25.5 -> 24.4 mm
- net /FLASH_SD2: track 16.5 -> 15.5 mm
Other:
- board text added: "BOOT"
- board text added: "RESET"
- board text added: "stav-keeb-60 v2a"
- board text removed: "stav-keeb-60 v0"
